Commit message: commit actuator section

File: Chapter6/Chapter6_ws/src/fishbot_description/urdf/fishbot/base.urdf.xacro (robot description, xacro)
@@ -1,4 +1,5 @@
 <?xml version="1.0"?>
 <robot xmlns:xacro="http://www.ros.org/wiki/xacro">
+    <link name="base_footprint" />
     <!-- base module -->
     <xacro:macro name="base_xacro" params="length radius">
@@ -20,4 +21,9 @@
             </visual>
         </link>
+        <joint name="joint_name" type="fixed">
+            <origin xyz="0.0 0.0 ${length/2.0+0.032-0.001}" rpy="0.0 0.0 0.0"/>
+            <parent link="base_footprint"/>
+            <child link="base_link"/>
+        </joint>
     </xacro:macro>
 </robot>

File: Chapter6/Chapter6_ws/src/fishbot_description/urdf/fishbot/fishbot.urdf.xacro (robot description, xacro)
@@ -7,7 +7,14 @@
 <xacro:include filename="$(find fishbot_description)/urdf/fishbot/sensor/camera.urdf.xacro"/>
 <xacro:include filename="$(find fishbot_description)/urdf/fishbot/sensor/laser.urdf.xacro"/>
+<!-- actuator_section -->
+<xacro:include filename="$(find fishbot_description)/urdf/fishbot/actuator/wheel.urdf.xacro"/>
+<xacro:include filename="$(find fishbot_description)/urdf/fishbot/actuator/caster.urdf.xacro"/>
 <xacro:base_xacro length="0.12" radius="0.10" />
 <xacro:imu_xacro xyz="0.0 0.0 0.02" />
 <xacro:camera_xacro xyz="0.10 0.0 0.075" />
 <xacro:laser_xacro xyz="0.0 0.0 0.10" />
+<xacro:wheel_xacro wheel_name="left_wheel" xyz="0 0.10 -0.06" />
+<xacro:wheel_xacro wheel_name="right_wheel" xyz="0 -0.10 -0.06" />
+<xacro:caster_xacro caster_name="front_caster" xyz="0.08 0.0 -0.076" />
+<xacro:caster_xacro caster_name="back_caster" xyz="-0.08 0.0 -0.076" />
 </robot>
