Commit message: commit collision

File: Chapter6/Chapter6_ws/src/fishbot_description/urdf/fishbot/actuator/caster.urdf.xacro (robot description, xacro)
@@ -17,4 +17,16 @@
                 </material>
             </visual>
+            <collision>
+                <!-- values of offset and rotation along its own geometric center -->
+                <origin xyz="0.0 0.0 0.0" rpy="0.0 0.0 0.0"/>
+                <!-- geometric shapes -->
+                <geometry>
+                    <sphere radius="0.016"/>
+                </geometry>
+                <!-- material -->
+                <material name="yellow">
+                    <color rgba="1.0 1.0 0.0 0.8"/>
+                </material>
+            </collision>
         </link>
         <!-- robot's joints, for assembling components of robot -->

File: Chapter6/Chapter6_ws/src/fishbot_description/urdf/fishbot/actuator/wheel.urdf.xacro (robot description, xacro)
@@ -17,4 +17,16 @@
                 </material>
             </visual>
+            <collision>
+                <!-- values of offset and rotation along its own geometric center -->
+                <origin xyz="0.0 0.0 0.0" rpy="1.57079 0.0 0.0"/>
+                <!-- geometric shapes -->
+                <geometry>
+                    <cylinder radius="0.032" length="0.04"/>
+                </geometry>
+                <!-- material -->
+                <material name="yellow">
+                    <color rgba="1.0 1.0 0.0 0.8"/>
+                </material>
+            </collision>
         </link>
         <!-- robot's joints, for assembling components of robot -->

File: Chapter6/Chapter6_ws/src/fishbot_description/urdf/fishbot/base.urdf.xacro (robot description, xacro)
@@ -20,4 +20,17 @@
                 </material>
             </visual>
+            <collision>
+                <!-- values of offset and rotation along its own geometric center -->
+                <origin xyz="0.0 0.0 0.0" rpy="0.0 0.0 0.0"/>
+                <!-- geometric shapes -->
+                <geometry>
+                    <!-- cylinder 0.10m*0.12m -->
+                    <cylinder radius="${radius}" length="${length}"/>
+                </geometry>
+                <!-- material -->
+                <material name="white">
+                    <color rgba="1.0 1.0 1.0 0.5"/>
+                </material>
+            </collision>
         </link>
         <joint name="joint_name" type="fixed">

File: Chapter6/Chapter6_ws/src/fishbot_description/urdf/fishbot/sensor/camera.urdf.xacro (robot description, xacro)
@@ -17,4 +17,16 @@
                 </material>
             </visual>
+            <collision>
+                <!-- values of offset and rotation along its own geometric center -->
+                <origin xyz="0.0 0.0 0.0" rpy="0.0 0.0 0.0"/>
+                <!-- geometric shapes -->
+                <geometry>
+                    <box size="0.02 0.10 0.02"/>
+                </geometry>
+                <!-- material -->
+                <material name="black">
+                    <color rgba="0.0 0.0 0.0 0.5"/>
+                </material>
+            </collision>
         </link>
         <!-- robot's joints, for assembling components of robot -->

File: Chapter6/Chapter6_ws/src/fishbot_description/urdf/fishbot/sensor/imu.urdf.xacro (robot description, xacro)
@@ -17,4 +17,16 @@
                 </material>
             </visual>
+            <collision>
+                <!-- values of offset and rotation along its own geometric center -->
+                <origin xyz="0.0 0.0 0.0" rpy="0.0 0.0 0.0"/>
+                <!-- geometric shapes -->
+                <geometry>
+                    <box size="0.02 0.02 0.02"/>
+                </geometry>
+                <!-- material -->
+                <material name="black">
+                    <color rgba="0.0 0.0 0.0 0.5"/>
+                </material>
+            </collision>
         </link>
         <!-- robot's joints, for assembling components of robot -->

File: Chapter6/Chapter6_ws/src/fishbot_description/urdf/fishbot/sensor/laser.urdf.xacro (robot description, xacro)
@@ -17,4 +17,16 @@
                 </material>
             </visual>
+            <collision>
+                <!-- values of offset and rotation along its own geometric center -->
+                <origin xyz="0.0 0.0 0.0" rpy="0.0 0.0 0.0"/>
+                <!-- geometric shapes -->
+                <geometry>
+                    <cylinder radius="0.01" length="0.10"/>
+                </geometry>
+                <!-- material -->
+                <material name="black">
+                    <color rgba="0.0 0.0 0.0 1.0"/>
+                </material>
+            </collision>
         </link>
         <!-- robot's LASER component -->
@@ -33,4 +45,16 @@
                 </material>
             </visual>
+            <collision>
+                <!-- values of offset and rotation along its own geometric center -->
+                <origin xyz="0.0 0.0 0.0" rpy="0.0 0.0 0.0"/>
+                <!-- geometric shapes -->
+                <geometry>
+                    <cylinder radius="0.02" length="0.02"/>
+                </geometry>
+                <!-- material -->
+                <material name="black">
+                    <color rgba="0.0 0.0 0.0 1.0"/>
+                </material>
+            </collision>
         </link>
         <!-- robot's joints, for assembling components of robot -->

Commit message: mass and inertia

File: Chapter6/Chapter6_ws/src/fishbot_description/urdf/fishbot/actuator/caster.urdf.xacro (robot description, xacro)
@@ -1,4 +1,5 @@
 <?xml version="1.0"?>
 <robot xmlns:xacro="http://www.ros.org/wiki/xacro">
+<xacro:include filename="$(find fishbot_description)/urdf/fishbot/common_inertia.xacro"/>
     <xacro:macro name="caster_xacro" params="caster_name xyz">
         <!-- robot's CASTER component -->
@@ -29,4 +30,5 @@
                 </material>
             </collision>
+            <xacro:sphere_inertia m="0.05" r="0.016" />
         </link>
         <!-- robot's joints, for assembling components of robot -->

File: Chapter6/Chapter6_ws/src/fishbot_description/urdf/fishbot/actuator/wheel.urdf.xacro (robot description, xacro)
@@ -1,4 +1,5 @@
 <?xml version="1.0"?>
 <robot xmlns:xacro="http://www.ros.org/wiki/xacro">
+<xacro:include filename="$(find fishbot_description)/urdf/fishbot/common_inertia.xacro"/>
     <xacro:macro name="wheel_xacro" params="wheel_name xyz">
         <!-- robot's WHEEL component -->
@@ -29,4 +30,5 @@
                 </material>
             </collision>
+            <xacro:cylinder_inertia m="0.05" r="0.032" h="0.04" />
         </link>
         <!-- robot's joints, for assembling components of robot -->

File: Chapter6/Chapter6_ws/src/fishbot_description/urdf/fishbot/base.urdf.xacro (robot description, xacro)
@@ -1,7 +1,8 @@
 <?xml version="1.0"?>
 <robot xmlns:xacro="http://www.ros.org/wiki/xacro">
-    <link name="base_footprint" />
+    <xacro:include filename="$(find fishbot_description)/urdf/fishbot/common_inertia.xacro"/>
     <!-- base module -->
     <xacro:macro name="base_xacro" params="length radius">
+        <link name="base_footprint" />
         <!-- Body Part of Robot -->
         <link name="base_link">
@@ -33,4 +34,5 @@
                 </material>
             </collision>
+            <xacro:cylinder_inertia m="1.0" r="${radius}" h="${length}" />
         </link>
         <joint name="joint_name" type="fixed">

File: Chapter6/Chapter6_ws/src/fishbot_description/urdf/fishbot/sensor/camera.urdf.xacro (robot description, xacro)
@@ -1,4 +1,5 @@
 <?xml version="1.0"?>
 <robot xmlns:xacro="http://www.ros.org/wiki/xacro">
+<xacro:include filename="$(find fishbot_description)/urdf/fishbot/common_inertia.xacro"/>
     <xacro:macro name="camera_xacro" params="xyz">
         <!-- robot's CAMERA component -->
@@ -29,4 +30,5 @@
                 </material>
             </collision>
+            <xacro:box_inertia m="0.1" w="0.02" h="0.10" d="0.02" />
         </link>
         <!-- robot's joints, for assembling components of robot -->

File: Chapter6/Chapter6_ws/src/fishbot_description/urdf/fishbot/sensor/imu.urdf.xacro (robot description, xacro)
@@ -1,4 +1,5 @@
 <?xml version="1.0"?>
 <robot xmlns:xacro="http://www.ros.org/wiki/xacro">
+<xacro:include filename="$(find fishbot_description)/urdf/fishbot/common_inertia.xacro"/>
     <xacro:macro name="imu_xacro" params="xyz">
         <!-- robot's IMU component -->
@@ -29,4 +30,5 @@
                 </material>
             </collision>
+            <xacro:box_inertia m="0.05" w="0.02" h="0.02" d="0.02" />
         </link>
         <!-- robot's joints, for assembling components of robot -->

File: Chapter6/Chapter6_ws/src/fishbot_description/urdf/fishbot/sensor/laser.urdf.xacro (robot description, xacro)
@@ -1,4 +1,5 @@
 <?xml version="1.0"?>
 <robot xmlns:xacro="http://www.ros.org/wiki/xacro">
+<xacro:include filename="$(find fishbot_description)/urdf/fishbot/common_inertia.xacro"/>
     <xacro:macro name="laser_xacro" params="xyz">
         <!-- laser cylinder component -->
@@ -29,4 +30,5 @@
                 </material>
             </collision>
+            <xacro:cylinder_inertia m="0.05" r="0.01" h="0.1" />
         </link>
         <!-- robot's LASER component -->
@@ -57,4 +59,5 @@
                 </material>
             </collision>
+            <xacro:cylinder_inertia m="0.10" r="0.02" h="0.02" />
         </link>
         <!-- robot's joints, for assembling components of robot -->

Commit message: add world and model

File: Chapter6/Chapter6_ws/src/fishbot_description/urdf/fishbot/actuator/caster.urdf.xacro (robot description, xacro)
@@ -39,4 +39,11 @@
             <axis xyz="0 1 0"/>
         </joint>
+        <gazebo reference="${caster_name}_link">
+            <mu1 value = "0.0"/>
+            <mu2 value = "0.0"/>
+            <kp value = "1000000000.0"/>
+            <kd value = "1.0"/>
+            <material> Gazebo/Yellow </material>
+        </gazebo>
     </xacro:macro>
 </robot>

File: Chapter6/Chapter6_ws/src/fishbot_description/urdf/fishbot/actuator/wheel.urdf.xacro (robot description, xacro)
@@ -39,4 +39,11 @@
             <axis xyz="0 1 0"/>
         </joint>
+        <gazebo reference="${wheel_name}_link">
+            <mu1 value = "20.0"/>
+            <mu2 value = "20.0"/>
+            <kp value = "1000000000.0"/>
+            <kd value = "1.0"/>
+            <material> Gazebo/Yellow </material>
+        </gazebo>
     </xacro:macro>
 </robot>

File: Chapter6/Chapter6_ws/src/fishbot_description/urdf/fishbot/sensor/camera.urdf.xacro (robot description, xacro)
@@ -38,4 +38,7 @@
             <origin xyz="${xyz}" rpy="0.0 0.0 0.0"/>
         </joint>
+        <gazebo reference="camera_link">
+            <material> Gazebo/Black </material>
+        </gazebo>
     </xacro:macro>
 </robot>

File: Chapter6/Chapter6_ws/src/fishbot_description/urdf/fishbot/sensor/imu.urdf.xacro (robot description, xacro)
@@ -38,4 +38,7 @@
             <origin xyz="${xyz}" rpy="0.0 0.0 0.0"/>
         </joint>
+        <gazebo reference="imu_link">
+            <material> Gazebo/Black </material>
+        </gazebo>
     </xacro:macro>
 </robot>

File: Chapter6/Chapter6_ws/src/fishbot_description/urdf/fishbot/sensor/laser.urdf.xacro (robot description, xacro)
@@ -72,4 +72,10 @@
             <origin xyz="${xyz}" rpy="0.0 0.0 0.0"/>
         </joint>
+        <gazebo reference="laser_cylinder_link">
+            <material> Gazebo/Black </material>
+        </gazebo>
+        <gazebo reference="laser_link">
+            <material> Gazebo/Black </material>
+        </gazebo>
     </xacro:macro>
 </robot>
